File: GatewayPlus_V1.4.kicad_pcb (KiCad board)
At the start: 2 copper layers, 100 x 60 mm, 276 parts, among them IC1 MP1584EN, IC2 MP1584EN, J1 SWD_LOG, J10 USB_OTG, J11 USB_WIFI, J2 LTDC_LCD_FPC_40p, J3 Micro_SD_Card, J4 ESP Anten, J5 LoRa_Anten, J6 HR911105A, J7 RS485, J8 Conn_Jack-DC, J9 AudioJack, Q1 BC847, Q2 BC847, SW1 SW_Push, SW2 ESP_RESET, SW3 ESP_BOOT, U1 STM32F429IGTx, U10 USBLC6-2SC6, U11 USBLC6-2SC6, U2 IS42S16400J - HY57V641620E, U3 ESP32-C3, U4 W25Q32JVSS, U5 SX1278, U6 MASWSS0192, U7 LAN8720A, U8 MAX485E, U9 ES8388, Y1 25MHz, Y2 40MHz, Y3 32MHz, Y4 25MHz, Y5 32.768KHz

Commit message: Finished Board.
Routing:
- net GND: vias 922 -> 914
Other:
- board text added: "AUDIO CODEC"
- board text removed: "CODEC"
Changed lines of the file:
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@@
     (effects (font (size 0.6 0.6) (thickness 0.15)) (justify left bottom))
   )
-  (gr_text "CODEC" (at 114 80.73) (layer "F.SilkS" knockout)
+  (gr_text "AUDIO CODEC" (at 109.94 80.74) (layer "F.SilkS" knockout)
     (effects (font (size 0.8 0.8) (thickness 0.2) bold) (justify left bottom))
   )
@@
   (via (at 109.52 121.06) (size 0.6) (drill 0.4) (layers "F.Cu" "B.Cu") (net 1))
   (via (at 141.66 76.05) (size 0.6) (drill 0.4) (layers "F.Cu" "B.Cu") (net 1))
-  (via (at 44.34 78.57) (size 0.6) (drill 0.4) (layers "F.Cu" "B.Cu") (net 1))
   (via (at 118.96 68.27) (size 0.6) (drill 0.4) (layers "F.Cu" "B.Cu") (net 1))
   (via (at 140.68 101.11) (size 0.6) (drill 0.4) (layers "F.Cu" "B.Cu") (net 1))
@@
   (via (at 132.83 96.68) (size 0.6) (drill 0.4) (layers "F.Cu" "B.Cu") (net 1))
   (via (at 126.73 96.69) (size 0.6) (drill 0.4) (layers "F.Cu" "B.Cu") (net 1))
-  (via (at 48.24 79.87) (size 0.6) (drill 0.4) (layers "F.Cu" "B.Cu") (net 1))
   (via (at 132.19 89.39) (size 0.6) (drill 0.4) (layers "F.Cu" "B.Cu") (net 1))
   (via (at 127.42 63.19) (size 0.6) (drill 0.4) (layers "F.Cu" "B.Cu") (net 1))
@@
   (via (at 62.56 91.63) (size 0.6) (drill 0.4) (layers "F.Cu" "B.Cu") (net 1))
   (via (at 94.35 61.77) (size 0.6) (drill 0.4) (layers "F.Cu" "B.Cu") (net 1))
-  (via (at 49.22 79.87) (size 0.6) (drill 0.4) (layers "F.Cu" "B.Cu") (net 1))
   (via (at 121.71 117.16) (size 0.5) (drill 0.3) (layers "F.Cu" "B.Cu") (net 1))
   (via (at 50.6 96.16) (size 0.6) (drill 0.4) (layers "F.Cu" "B.Cu") (net 1))
@@
   (via (at 83.72 99.57) (size 0.6) (drill 0.4) (layers "F.Cu" "B.Cu") (net 1))
   (via (at 44.34 69.57) (size 0.6) (drill 0.4) (layers "F.Cu" "B.Cu") (net 1))
-  (via (at 50.16 79.87) (size 0.6) (drill 0.4) (layers "F.Cu" "B.Cu") (net 1))
   (via (at 87.28 116.39) (size 0.6) (drill 0.4) (layers "F.Cu" "B.Cu") (net 1))
   (via (at 124.7 103.54) (size 0.6) (drill 0.4) (layers "F.Cu" "B.Cu") (net 1))
@@
   (via (at 127.15 81) (size 0.6) (drill 0.4) (layers "F.Cu" "B.Cu") (net 1))
   (via (at 52.52 96.16) (size 0.6) (drill 0.4) (layers "F.Cu" "B.Cu") (net 1))
-  (via (at 45.55 78.57) (size 0.6) (drill 0.4) (layers "F.Cu" "B.Cu") (net 1))
   (via (at 127.7 87.63) (size 0.5) (drill 0.3) (layers "F.Cu" "B.Cu") (free) (net 1))
   (via (at 131.43 66.75) (size 0.6) (drill 0.4) (layers "F.Cu" "B.Cu") (net 1))
@@
   (via (at 57.49 72.36) (size 0.6) (drill 0.4) (layers "F.Cu" "B.Cu") (net 1))
   (via (at 133.99 96.69) (size 0.6) (drill 0.4) (layers "F.Cu" "B.Cu") (net 1))
-  (via (at 45.55 79.55) (size 0.6) (drill 0.4) (layers "F.Cu" "B.Cu") (net 1))
   (via (at 47.74 94.95) (size 0.6) (drill 0.4) (layers "F.Cu" "B.Cu") (net 1))
   (via (at 49.21 86.26) (size 0.6) (drill 0.4) (layers "F.Cu" "B.Cu") (net 1))
@@
   (via (at 78.14 103.27) (size 0.6) (drill 0.4) (layers "F.Cu" "B.Cu") (net 1))
   (via (at 106.03 69.82) (size 0.6) (drill 0.4) (layers "F.Cu" "B.Cu") (net 1))
-  (via (at 44.34 79.55) (size 0.6) (drill 0.4) (layers "F.Cu" "B.Cu") (net 1))
   (via (at 93.07 121.06) (size 0.6) (drill 0.4) (layers "F.Cu" "B.Cu") (net 1))
   (via (at 126.62 92.93) (size 0.6) (drill 0.4) (layers "F.Cu" "B.Cu") (net 1))
   (via (at 132.3 109.64) (size 0.6) (drill 0.4) (layers "F.Cu" "B.Cu") (net 1))
-  (via (at 47.24 79.87) (size 0.6) (drill 0.4) (layers "F.Cu" "B.Cu") (net 1))
   (via (at 52.07 85.05) (size 0.6) (drill 0.4) (layers "F.Cu" "B.Cu") (net 1))
   (via (at 106.35 61.77) (size 0.6) (drill 0.4) (layers "F.Cu" "B.Cu") (net 1))
