File: MicroSD.kicad_sch (KiCad schematic)
At the start: 6 parts, among them J3 Micro_SD_Card

Commit message: Finish board.
Parts:
- J3: footprint Anh_Footprints:MicroSD_Socket -> Anh_Footprints:MicroSD_Socket_9P
Changed lines of the file:
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@@
       (effects (font (size 1.27 1.27)))
     )
-    (property "Footprint" "Anh_Footprints:MicroSD_Socket" (at 153.67 55.88 0)
+    (property "Footprint" "Anh_Footprints:MicroSD_Socket_9P" (at 153.67 55.88 0)
       (effects (font (size 1.27 1.27)) hide)
     )
